File: vca-adsr.kicad_pcb (KiCad board)
At the start: 2 copper layers, 65 x 75 mm, 82 parts, among them Q1 2N3904, Q2 2N3904, Q3 2N3904, U1 TL074, U2 7555, U3 TL072

Commit message: Fix envelope trigger
Parts:
- added R27: 1M, Resistor_THT:R_Axial_DIN0207_L6.3mm_D2.5mm_P2.54mm_Vertical, F.Cu at (130.5, 93.1)
- added R28: 100k, Resistor_THT:R_Axial_DIN0207_L6.3mm_D2.5mm_P2.54mm_Vertical, F.Cu at (126.2, 96.1)
- R4, R5: footprint Resistor_THT:R_Axial_DIN0207_L6.3mm_D2.5mm_P7.62mm_Horizontal -> Resistor_THT:R_Axial_DIN0207_L6.3mm_D2.5mm_P2.54mm_Vertical
- renumbered Q1 to Q1*1, Q2 to Q2*1
Routing:
- net -12V: track 111.0 -> 138.2 mm
- net Net-(D3-Pad1): track 6.31 -> 13.3 mm
- net Net-(R27-Pad2): track 4.90 -> 8.49 mm
- net Net-(C1-Pad2): track 44.2 -> 45.3 mm
